Commit message: edited some files

File: major_snakebot_description/urdf/major_snakebot.xacro (robot description, xacro)
@@ -156,5 +156,5 @@
 </joint>
 <joint name="lidar_joint" type="fixed">
-  <origin xyz="0.0 -0.008 -0.01" rpy="0 0 -1.57"/>
+  <origin xyz="0.0 -0.008 -0.01" rpy="0 0 -1.80"/>
   <parent link="base_link"/>
   <child link="lidar_1"/>
